File: device/KiCad/piclodio3/piclodio3.sch (KiCad schematic (older format))
At the start: 18 parts, among them J3 40HAT, J6 CONN_02X02, J9 CONN_01X02, Q1 DMG2305UX, Q2 DMMT5401, U2 CAT24C32

Commit message: Remove useless components
Parts:
- removed J6: CONN_02X02, Connector_PinHeader_2.54mm:PinHeader_2x02_P2.54mm_Vertical, symbol Connector_Generic:Conn_02x02_Odd_Even
- removed Q1: DMG2305UX, Package_TO_SOT_SMD:SOT-23, symbol raspberrypi_hat:DMG2305UX
- removed Q2: DMMT5401, Package_TO_SOT_SMD:SOT-23-6, symbol raspberrypi_hat:DMMT5401
- removed R11, R7, R9: DNP, Resistor_SMD:R_0603_1608Metric_Pad0.84x1.00mm_HandSolder, symbol Device:R
- removed R23: 10K, Resistor_SMD:R_0603_1608Metric_Pad0.84x1.00mm_HandSolder, symbol Device:R
- removed R24: 47K, Resistor_SMD:R_0603_1608Metric_Pad0.84x1.00mm_HandSolder, symbol Device:R
Other:
- note removed: "5V Powered HAT Protection"
- note removed: "FLEXIBLE POWER SELECTION"
- note removed: "HAT spec indicates to NEVER\npower the 3.3V pins on the Raspberry Pi \nfrom the HAT header. Only connect the 3.3V\npower from the Pi if the HAT does not have\n3.3V on board.\n\nIF you are designing a board that could\neither be powered by the Pi or from the HAT\nthe jumpers here can be used.\n\nIn most cases, either design the HAT \nto provide the 5V to the Pi and use the\nprotection circuit abov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"
- note removed: "This is the recommended 5V rail protection for \na HAT with power going to the Pi.\nSee https://github.com/raspberrypi/hats/blob/master/designguide.md#back-powering-the-pi-via-the-j8-gpio-header"
- moved on the sheet: H1, H2, H3, H4, J3, J9, R29, R6, R8, U2
